File: kicad/carte-capteur.sch (KiCad schematic (older format))
At the start: 33 parts, among them J1 PDB, J2 PWR_IN, J3 PROG, J4 Fix, J5 Fix, J6 Fix, J7 Fix, J8 I2C, J9 I2C, U1 PIC24FJ128GA202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

Commit message: Association empreintes
Parts:
- D3: footprint (none) -> LEDs:LED_D3.0mm
- J8, J9: footprint (none) -> Epsa:KK_2C
- R4, R5, R6: footprint (none) -> Resistors_THT:R_Axial_DIN0204_L3.6mm_D1.6mm_P7.62mm_Horizontal
- U1: footprint (none) -> Housings_DIP:DIP-28_W7.62mm
- U2, U3: footprint (none) -> conn_shield:conn_shield
Changed lines of the file:
@@
 F 0 "U1" V 2350 1300 60  0000 C CNN
 F 1 "PIC24FJ128GA202" V 2250 1200 60  0000 C CNN
-F 2 "" H 2300 1300 60  0001 C CNN
+F 2 "Housings_DIP:DIP-28_W7.62mm" H 2300 1300 60  0001 C CNN
 F 3 "" H 2300 1300 60  0001 C CNN
 	1    2300 1300
@@
 F 0 "D3" H 3500 3100 50  0000 C CNN
 F 1 "GREEN" H 3500 2900 50  0000 C CNN
-F 2 "" H 3500 3000 50  0001 C CNN
+F 2 "LEDs:LED_D3.0mm" H 3500 3000 50  0001 C CNN
 F 3 "" H 3500 3000 50  0001 C CNN
 	1    3500 3000
@@
 F 0 "R4" V 3580 2650 50  0000 C CNN
 F 1 "470" V 3500 2650 50  0000 C CNN
-F 2 "" V 3430 2650 50  0001 C CNN
+F 2 "Resistors_THT:R_Axial_DIN0204_L3.6mm_D1.6mm_P7.62mm_Horizontal" V 3430 2650 50  0001 C CNN
 F 3 "" H 3500 2650 50  0001 C CNN
 	1    3500 2650
@@
 F 0 "R6" V 7030 1500 50  0000 C CNN
 F 1 "10k" V 6950 1500 50  0000 C CNN
-F 2 "" V 6880 1500 50  0001 C CNN
+F 2 "Resistors_THT:R_Axial_DIN0204_L3.6mm_D1.6mm_P7.62mm_Horizontal" V 6880 1500 50  0001 C CNN
 F 3 "" H 6950 1500 50  0001 C CNN
 	1    6950 1500
@@
 F 0 "R5" V 7030 1100 50  0000 C CNN
 F 1 "10k" V 6950 1100 50  0000 C CNN
-F 2 "" V 6880 1100 50  0001 C CNN
+F 2 "Resistors_THT:R_Axial_DIN0204_L3.6mm_D1.6mm_P7.62mm_Horizontal" V 6880 1100 50  0001 C CNN
 F 3 "" H 6950 1100 50  0001 C CNN
 	1    6950 1100
@@
 F 0 "J9" H 6050 3200 50  0000 C CNN
 F 1 "I2C" H 6050 2900 50  0000 C CNN
-F 2 "" H 6050 3100 50  0001 C CNN
+F 2 "Epsa:KK_2C" H 6050 3100 50  0001 C CNN
 F 3 "" H 6050 3100 50  0001 C CNN
 	1    6050 3100
@@
 F 0 "J8" H 5650 3200 50  0000 C CNN
 F 1 "I2C" H 5650 2900 50  0000 C CNN
-F 2 "" H 5650 3100 50  0001 C CNN
+F 2 "Epsa:KK_2C" H 5650 3100 50  0001 C CNN
 F 3 "" H 5650 3100 50  0001 C CNN
 	1    5650 3100
@@
 F 0 "U2" H 7750 2300 60  0000 C CNN
 F 1 "Shield_gauche" H 7600 2400 60  0000 C CNN
-F 2 "" H 7750 2300 60  0001 C CNN
+F 2 "conn_shield:conn_shield" H 7750 2300 60  0001 C CNN
 F 3 "" H 7750 2300 60  0001 C CNN
 	1    7750 2300
@@
 F 0 "U3" H 8300 2300 60  0000 C CNN
 F 1 "Shield_droit" H 8200 2400 60  0000 C CNN
-F 2 "" H 8300 2300 60  0001 C CNN
+F 2 "conn_shield:conn_shield" H 8300 2300 60  0001 C CNN
 F 3 "" H 8300 2300 60  0001 C CNN
 	1    8300 2300
